File: hardware/carvera_PCB/FARESHARE KICAD/_autosave-FARESHARE KICAD.kicad_pcb (KiCad board)
At the start: 2 copper layers, 14 parts, among them J1 0022232041, J2 0022232041, J3 0022232041, J4 22-23-2021, J5 PJ-102A

Commit message: PCb design and gerber files generated
Parts:
- removed the R2 at (105.4, 81.1)
- removed R3: 1M, SparkFun-Resistor:R_0402_1005Metric
- added A3: Arduino_UNO_R2, Module:Arduino_UNO_R2, F.Cu at (109.3, 51.7)
- added R2: R, Resistor_THT:R_Axial_DIN0207_L6.3mm_D2.5mm_P7.62mm_Horizontal, F.Cu at (147.3, 76.2)
- added R2: 0.47, SparkFun-Resistor:R_0603_1608Metric, F.Cu at (1.50, 0.76)
- R1: value 1M -> R; footprint SparkFun-Resistor:R_0402_1005Metric -> Resistor_THT:R_Axial_DIN0207_L6.3mm_D2.5mm_P7.62mm_Horizontal
- moved J5 43.7 mm to (92.5, 56.5), turned to 90 degrees
- moved J4 41.4 mm to (139.7, 86.5)
- moved J2 41.4 mm to (106.7, 73.7)
- moved A1 39.6 mm to (98.2, 83.8)
- moved R1 37.8 mm to (142.2, 71.1), turned to -90 degrees
- moved C2 36.8 mm to (104.0, 61.0)
- moved J1 32.1 mm to (134.5, 64.2)
- moved A2 31.9 mm to (126.8, 76.9)
- moved J3 30.6 mm to (125.0, 87.0), turned to 0 degrees
- moved C1 20.8 mm to (133.5, 56.5), turned to -90 degrees
- moved S1 16.5 mm to (112.8, 92.2), turned to 90 degrees
- moved S2 11.9 mm to (103.0, 93.5), turned to 180 degrees
Connections:
- A1 pad 15: D10 -> D12
- A1 pad 16: D11 -> D13
- J4 pad 2: D2 -> D3
- R1 pad 1: D4 -> D5
- R1 pad 2: D5 -> D4
- S1 pad 3: D13 -> D10
- S2 pad 3: D12 -> D11
Routing:
- net +5V: track 0.00 -> 76.0 mm
- net +12V: track 0.00 -> 47.0 mm
- net D12: track 0.00 -> 37.6 mm
- net D13: track 0.00 -> 35.5 mm
- net D5: track 0.00 -> 33.1 mm
- net D8: track 0.00 -> 29.3 mm
- net D3: track 0.00 -> 28.1 mm
- net D9: track 0.00 -> 25.7 mm
- net D2: track 0.00 -> 19.3 mm
- net D11: track 0.00 -> 16.9 mm
- net D4: track 0.00 -> 15.6 mm
- net D7: track 0.00 -> 13.9 mm
- net D6: track 0.00 -> 13.9 mm
- net Net-(A1-VMOT): track 0.00 -> 10.8 mm
- net Net-(A1-2A): track 0.00 -> 9.53 mm
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- added copper zone on B.Cu, net GND
- added copper zone on F.Cu, net GND
Other:
- board outline added: 70 x 54 mm
