File: hardware/carvera_PCB/FARESHARE KICAD/_autosave-FARESHARE KICAD.kicad_pcb (KiCad board)
At the start: 2 copper layers, 70 x 55 mm, 14 parts, among them J1 0022232041, J2 0022232041, J3 0022232041, J4 22-23-2021, J5 Barrel_Jack_Switch_Pin3Ring

Commit message: barrel jack updated to a round one
Parts:
- J5: footprint Connector_BarrelJack:BarrelJack_Horizontal -> Connector_BarrelJack:BarrelJack_Wuerth_694102107102_1.0x3.9mm
- moved J5 15.5 mm to (81.8, 57.0), turned to -90 degrees

Commit message: Traces changed and other files updated accordingly
Parts:
- A1, A2: moved to B.Cu
- J5: footprint Connector_BarrelJack:BarrelJack_Wuerth_694102107102_1.0x3.9mm -> Connector_BarrelJack:BarrelJack_CUI_PJ-102AH_Horizontal
- moved R1 29.4 mm to (125.5, 95.3), turned to 90 degrees
- moved S2 20.9 mm to (85.8, 81.8), turned to 0 degrees
- moved J2 18.0 mm to (90.0, 67.0)
- moved S1 16.5 mm to (122.2, 78.8), turned to 0 degrees
- moved C1 14.0 mm to (119.5, 56.5)
- moved J5 13.7 mm to (95.5, 56.5)
- moved J3 12.5 mm to (113.8, 92.5), turned to 180 degrees
- moved R2 12.1 mm to (143.5, 87.7)
- moved J4 9.62 mm to (131.2, 91.0)
- moved A2 9.08 mm to (133.7, 82.9), turned to 0 degrees
- moved J1 8.59 mm to (126.0, 65.4)
- moved C2 5.67 mm to (107.5, 56.5), turned to -90 degrees
- moved A1 1.72 mm to (99.8, 83.2), turned to 0 degrees
Connections:
- A1 pad 15: D12 -> D11
- A1 pad 16: D13 -> D12
- A2 pad 15: D8 -> D7
- A2 pad 16: D9 -> D8
- J3 pad 1: D7 -> D9
- J3 pad 2: D6 -> D10
- J4 pad 1: D4 -> D5
- J4 pad 2: D3 -> D4
- R1 pad 1: D5 -> D6
- R1 pad 2: D4 -> D5
- R2 pad 1: D3 -> D4
- S1 pad 3: D10 -> D3
- S2 pad 3: D11 -> D10
Routing:
- net D12: track 37.6 -> 0.00 mm
- net D13: track 35.5 -> 0.00 mm
- net D5: track 33.1 -> 0.00 mm
- net D8: track 29.3 -> 0.00 mm
- net D3: track 28.1 -> 0.00 mm
- net D9: track 25.7 -> 0.00 mm
- net D4: track 25.0 -> 0.00 mm
- net D2: track 19.3 -> 0.00 mm
- net D11: track 16.9 -> 0.00 mm
- net D7: track 13.9 -> 0.00 mm
- net D6: track 13.9 -> 0.00 mm
- net +12V: track 47.3 -> 35.5 mm
- net Net-(A2-VMOT): track 6.91 -> 16.3 mm
- net D10: track 8.03 -> 0.00 mm
- net +5V: track 133.0 -> 126.5 mm
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