File: hardware/carvera_PCB/FARESHARE KICAD/_autosave-FARESHARE KICAD.kicad_sch (KiCad schematic)
At the start: 14 parts, among them J1 0022232041, J2 0022232041, J3 0022232041, J4 22-23-2021, J5 PJ-102A

Commit message: circuit components added
Parts:
- added A3: Arduino_Uno_R1_Shield, PCM_arduino-library:Arduino_Uno_R2_Shield, symbol arduino-library:Arduino_Uno_R1_Shield
Connections:
- net GND: now reaches A1.1 (GND)
- net GND: now also A1.7 (GND)
- net at A1.3 (1B): now also J2.4
- net at A1.4 (1A): now also J2.3
- net at A1.5 (2A): now also J2.2
- net at A1.6 (2B): now also J2.1
- net at J1.1: now also A2.6 (2B)
- net at J1.2: now also A2.5 (2A)
- net at J1.3: now also A2.4 (1A)
- net at J1.4: now also A2.3 (1B)
Other:
- company: (none) -> Sussex university
- title: (none) -> Fareshare
- moved on the sheet: A1, A2, C1, C2, J1, J2, J3, J4, J5, R1, R3, S1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

Commit message: Kicad files updated
Parts:
- removed S1, S2: KS-01Q-01_Obsolete, digikey-footprints:PushButton_Round_D12mm_THT_KS-01Q-01, symbol dk_Pushbutton-Switches:KS-01Q-01_Obsolete
- added S1, S2: 1825910-6, digikey-footprints:Switch_Tactile_THT_6x6mm, symbol dk_Tactile-Switches:1825910-6
- C1, C2: footprint ~ -> Capacitor_THT:CP_Radial_D5.0mm_P2.00mm
Connections:
- net GND: now also A2.1 (GND), A2.7 (GND), A3.GND1 (GND), A3.GND2 (GND), A3.GND3 (GND), J3.4, J5.2, J5.3, S1.4, S2.4
- net +5V: now reaches A3.5V1 (5V)
- net +5V: now also A1.2 (VDD), A2.2 (VDD), J3.3
- net D10: now reaches A3.D10 (D10_CS)
- net D10: now also A1.15 (STEP)
- net D11: now reaches A3.D11
- net D11: now also A1.16 (DIR)
- net D12: now reaches A3.D12
- net D12: now also S2.3
- net D13: now reaches A3.D13
- net D13: now also S1.3
- net D2: now reaches A3.D2 (D2_INT0)
- net D2: now also J4.2, R3.2
- net D3: now reaches A3.D3 (D3_INT1)
- net D3: now also R3.1
- net D4: now reaches A3.D4
- net D4: now also J4.1, R1.1
- net D5: now reaches A3.D5
- net D5: now also R1.2
- net D6: now reaches A3.D6
- net D6: now also J3.2
- net D7: now reaches A3.D7
- net D7: now also J3.1
- net D8: now reaches A3.D8
- net D8: now also A2.15 (STEP)
- net D9: now reaches A3.D9
- net D9: now also A2.16 (DIR)
- net +12V: now reaches A3.VIN
- net +12V: now also C1.1, C2.1, J5.1
- net at C1.2: now also A2.8 (VMOT)
- net at C2.2: now also A1.8 (VMOT)
- net at A1.13 (~{RESET}): now also A1.14 (~{SLEEP})
- net at A2.13 (~{RESET}): now also A2.14 (~{SLEEP})
Other:
- company: Sussex university -> (none)
- title: Fareshare -> (none)
- moved on the sheet: A1, A2, C1, C2, J1, J2, J3, J4, J5, R1, R3

Commit message: PCb design and gerber files generated
Parts:
- removed A3: Arduino_Uno_R1_Shield, PCM_arduino-library:Arduino_Uno_R2_Shield, symbol arduino-library:Arduino_Uno_R1_Shield
- removed R1, R3: 1M, SparkFun-Resistor:R_0402_1005Metric, symbol SparkFun-Resistor:1M_0402
- removed R2: 180, SparkFun-Resistor:R_0603_1608Metric, symbol SparkFun-Resistor:180_0603
- added A3: Arduino_UNO_R2, Module:Arduino_UNO_R2, symbol MCU_Module:Arduino_UNO_R2
- added R1, R2: R, Resistor_THT:R_Axial_DIN0207_L6.3mm_D2.5mm_P7.62mm_Horizontal, symbol device:R
Connections:
- net +12V: now also A3.8 (VIN)
- net +5V: now also A3.5 (+5V)
- net D10: now also S1.3, A3.25 (D10); no longer A1.15 (STEP)
- net D11: now also S2.3, A3.26 (D11); no longer A1.16 (DIR)
- net D12: now also A1.15 (STEP), A3.27 (D12); no longer S2.3
- net D13: now also A1.16 (DIR), A3.28 (D13); no longer S1.3
- net D2: now also A3.17 (D2), R2.2; no longer J4.2
- net D3: now also J4.2, A3.18 (D3), R2.1
- net D4: now also A3.19 (D4), R1.2
- net D5: now also A3.20 (D5), R1.1
- net D6: now also A3.21 (D6)
- net D7: now also A3.22 (D7)
- net D8: now also A3.23 (D8)
- net D9: now also A3.24 (D9)
- net GND: now also A3.29 (GND), A3.6 (GND), A3.7 (GND)
Other:
- company: (none) -> Sussex University
- title: (none) -> FARESHARE
