File: hardware/carvera_PCB/FARESHARE KICAD/_autosave-FARESHARE KICAD.kicad_sch (KiCad schematic)
At the start: 14 parts, among them J1 0022232041, J2 0022232041, J3 0022232041, J4 22-23-2021, J5 Barrel_Jack_Switch_Pin3Ring

Commit message: Traces changed and other files updated accordingly
Parts:
- J5: footprint Connector_BarrelJack:BarrelJack_Horizontal -> Connector_BarrelJack:BarrelJack_CUI_PJ-102AH_Horizontal
Connections:
- net D10: now also A1.16 (DIR); no longer S1.3
- net D11: now also J3.1; no longer S2.3
- net D12: now also J3.2; no longer A1.15 (STEP)
- net D13: now also S2.3; no longer A1.16 (DIR)
- net D3: now also A2.15 (STEP); no longer J4.2, R2.1
- net D4: now also A2.16 (DIR); no longer J4.1, R1.2
- net D5: now also J4.2, R2.1; no longer R1.1
- net D6: now also J4.1, R1.2; no longer J3.2
- net D7: now also R1.1; no longer J3.1
- net D8: now also S1.3; no longer A2.15 (STEP)
- net D9: now also A1.15 (STEP); no longer A2.16 (DIR)

Commit message: trying to use edge cut to cut slots
Connections:
- net D2: now also A2.16 (DIR); no longer R2.2
- net D4: now also R2.2; no longer A2.16 (DIR)
Changed lines of the file:
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@@
 		)
 	)
-	(global_label "D4"
+	(global_label "D2"
 		(shape input)
 		(at 214.63 64.77 180)
@@
 		)
 	)
-	(global_label "D2"
+	(global_label "D4"
 		(shape input)
 		(at 256.54 118.11 0)

Commit message: Will vias work?
Parts:
- J5: footprint Connector_BarrelJack:BarrelJack_CUI_PJ-102AH_Horizontal -> Connector_BarrelJack:BarrelJack_GCT_DCJ200-10-A_Horizontal
Changed lines of the file:
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@@
 			)
 		)
-		(property "Footprint" "Connector_BarrelJack:BarrelJack_CUI_PJ-102AH_Horizontal"
+		(property "Footprint" "Connector_BarrelJack:BarrelJack_GCT_DCJ200-10-A_Horizontal"
 			(at 52.07 51.816 0)
 			(effects
